File: mcu.kicad_sch (KiCad schematic)
At the start: 25 parts

Commit message: PCB Routing is done for first Proto
Parts:
- removed D?: LED_HeartBeat, LED_SMD:LED_0603_1608Metric, symbol Device:LED_Small
- removed FB?: 180 @ 100 Mhz, Inductor_SMD:L_0603_1608Metric_Pad1.05x0.95mm_HandSolder, symbol Device:FerriteBead_Small
- removed R?: 1.5k, Resistor_SMD:R_0402_1005Metric, symbol Device:R_Small
- added R6, R8: 0R, Resistor_SMD:R_0402_1005Metric, symbol Device:R_Small
- C3, C5: renamed from C?; footprint Capacitor_Tantalum_SMD:CP_EIA-3216-18_Kemet-A -> Capacitor_Tantalum_SMD:CP_EIA-3216-18_Kemet-A_Pad1.58x1.35mm_HandSolder
- J4: renamed from J?; footprint (none) -> Connector_USB:USB_C_Receptacle_HRO_TYPE-C-31-M-12
- R10: renamed from R?; value 82K -> 1.5K; footprint (none) -> Resistor_SMD:R_0402_1005Metric
- R11, R13: renamed from R?; footprint (none) -> Resistor_SMD:R_0402_1005Metric
- R12: renamed from R?; value 33K -> 1K; footprint (none) -> Resistor_SMD:R_0402_1005Metric
- gave numbers to parts that had none: 15
Connections:
- net USB_VBUS_DET: now also R8.1; no longer R10.2, R12.1
- net Vdda: now also R6.2
- net +3V3 renamed +3.3V
- net +3.3V: now also R6.1
- new net: R10.2, R12.1, R8.2
- no-connect marks 30 -> 31
Other:
- moved on the sheet: C3, C4, C5, C6, C7, C8, C9, R3, R4, SW1
