File: power.kicad_sch (KiCad schematic)
At the start: 5 parts

Commit message: PCB Routing is done for first Proto
Parts:
- added C2: 10uF, Capacitor_Tantalum_SMD:CP_EIA-3216-18_Kemet-A_Pad1.58x1.35mm_HandSolder, symbol Device:C_Polarized_Small
- added R14: 0R, Resistor_SMD:R_0402_1005Metric, symbol Device:R_Small
- added TP2: TP_MCU_PWR, TestPoint:TestPoint_Pad_D2.0mm, symbol Connector:TestPoint_Probe
- added U1: AMS1117-3.3, Package_TO_SOT_SMD:SOT-223-3_TabPin2, symbol Regulator_Linear:AMS1117-3.3
- C1: renamed from C?; footprint (none) -> Capacitor_Tantalum_SMD:CP_EIA-3216-18_Kemet-A_Pad1.58x1.35mm_HandSolder
- J1: renamed from J?; footprint (none) -> Connector_USB:USB_C_Receptacle_HRO_TYPE-C-31-M-12
- R1, R2: renamed from R?; footprint (none) -> Resistor_SMD:R_0402_1005Metric
- TP1: renamed from TP?; footprint (none) -> TestPoint:TestPoint_Pad_D2.0mm
Connections:
- net +5V: now also U1.3 (VI)
- net Earth: now also R14.2
- net GND: now also C2.2, R14.1, U1.1 (GND)
- new net +3.3V: C2.1, TP2.1, U1.2 (VO)
Other:
- moved on the sheet: C1, J1, R1, R2, TP1
